Commit message: fix joint_states

File: telekinesis/telekinesis/orca_hand/orcahand_right_wrist_fixed.urdf (robot description, URDF)
Before this commit: robot orcahand_right, 42 links, 41 joints
Joints:
- joint right_thumb_abd: limit lower=-1.08211 upper=0.0 effort=100 velocity=100 -> lower=-1.08211 upper=1 effort=100 velocity=100
